File: Glasses.sch (EAGLE design)
At the start: 190 parts, among them U1 APA1022020, U10 APA1022020, U100 APA1022020, U101 APA1022020, U102 APA1022020, U103 APA1022020, U104 APA1022020, U105 APA1022020, U106 APA1022020, U107 APA1022020, U108 APA1022020, U109 APA1022020, U11 APA1022020, U110 APA1022020, U111 APA1022020, U112 APA1022020, U113 APA1022020, U114 APA1022020, U115 APA1022020, U116 APA1022020, U117 APA1022020, U118 APA1022020, U119 APA1022020, U12 APA1022020, U120 APA1022020, U121 APA1022020, U122 APA1022020, U123 APA1022020, U124 APA1022020, U125 APA1022020, U126 APA1022020, U127 APA1022020, U128 APA1022020, U129 APA1022020, U13 APA1022020, U130 APA1022020, U131 APA1022020, U132 APA1022020, U133 APA1022020, U134 APA1022020, U135 APA1022020, U136 APA1022020, U137 APA1022020, U138 APA1022020, U139 APA1022020, U14 APA1022020, U140 APA1022020, U141 APA1022020, U142 APA1022020, U143 APA1022020, U144 APA1022020, U145 APA1022020, U146 APA1022020, U147 APA1022020, U148 APA1022020, U149 APA1022020, U15 APA1022020, U150 APA1022020, U151 APA1022020, U152 APA1022020, U153 APA1022020, U154 APA1022020, U155 APA1022020, U156 APA1022020, U157 APA1022020, U158 APA1022020, U159 APA1022020, U16 APA1022020, U160 APA1022020, U161 APA1022020, U162 APA1022020, U163 APA1022020, U164 APA1022020, U165 APA1022020, U166 APA1022020, U167 APA1022020, U168 APA1022020, U169 APA1022020, U17 APA1022020, U170 APA1022020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

Commit message: laid out footpirnts, routing needed
Parts:
- added J1, J2: (no value), SparkFun-Connectors:QWIIC_CONNECTORJS-1MM
- added U191, U192, U193, U194, U195, U196, U197, U198, U199, U200, U201, U202, U203, U204, U205, U206, U207, U208, U209, U210, U211, U212, U213, U214, U215, U216, U217, U218, U219, U220, U221, U222, U223, U224, U225, U226, U227, U228, U229, U230, U231, U232, U233, U234, U235, U236, U237, U238, U239, U240, U241, U242, U243, U244, U245, U246, U247, U248, U249, U250, U251, U252: APA1022020, 1_BES_Optoelectronics:APA1022020
Connections:
- new net CK7: U196.CO, U197.CI
- new net CK8: U224.CO, U225.CI
- new net N$365: U190.CO, U191.CI
- new net N$366: U190.DO, U191.DI
- new net N$367: U191.CO, U192.CI
- new net N$368: U191.DO, U192.DI
- new net N$369: U192.DO, U193.DI
- new net N$370: U192.CO, U193.CI
- new net N$371: U193.CO, U194.CI
- new net N$372: U193.DO, U194.DI
- new net N$373: U194.CO, U195.CI
- new net N$374: U194.DO, U195.DI
- new net N$379: U195.CO, U196.CI
- new net N$380: U195.DO, U196.DI
- new net N$381: U197.DO, U198.DI
- new net N$382: U197.CO, U198.CI
- new net N$383: U198.CO, U199.CI
- new net N$384: U198.DO, U199.DI
- new net N$385: U199.DO, U200.DI
- new net N$386: U199.CO, U200.CI
- new net N$387: U200.CO, U201.CI
- new net N$388: U200.DO, U201.DI
- new net N$389: U201.CO, U202.CI
- new net N$390: U201.DO, U202.DI
- new net N$391: U202.CO, U203.CI
- new net N$392: U202.DO, U203.DI
- new net N$393: U204.DO, U205.DI
- new net N$394: U204.CO, U205.CI
- new net N$395: U205.CO, U206.CI
- new net N$396: U205.DO, U206.DI
- new net N$397: U206.DO, U207.DI
- new net N$398: U206.CO, U207.CI
- new net N$399: U207.CO, U208.CI
- new net N$400: U207.DO, U208.DI
- new net N$401: U208.CO, U209.CI
- new net N$402: U208.DO, U209.DI
- new net N$403: U209.CO, U210.CI
- new net N$404: U209.DO, U210.DI
- new net N$405: U203.DO, U204.DI
- new net N$406: U203.CO, U204.CI
- new net N$407: U211.DO, U212.DI
- new net N$408: U211.CO, U212.CI
- new net N$409: U212.CO, U213.CI
- new net N$410: U212.DO, U213.DI
- new net N$411: U213.DO, U214.DI
- new net N$412: U213.CO, U214.CI
- new net N$413: U214.CO, U215.CI
- new net N$414: U214.DO, U215.DI
- new net N$415: U215.CO, U216.CI
- new net N$416: U215.DO, U216.DI
- new net N$417: U216.CO, U217.CI
- new net N$418: U216.DO, U217.DI
- new net N$419: U217.DO, U218.DI
- new net N$420: U217.CO, U218.CI
- new net N$421: U210.DO, U211.DI
- new net N$422: U210.CO, U211.CI
- new net N$423: U219.DI
- new net N$424: U219.CI
- new net N$425: U219.CO, U220.CI
- new net N$426: U219.DO, U220.DI
- new net N$427: U220.DO, U221.DI
- new net N$428: U220.CO, U221.CI
- new net N$429: U221.CO, U222.CI
- new net N$430: U221.DO, U222.DI
- new net N$431: U222.CO, U223.CI
- new net N$432: U222.DO, U223.DI
- new net N$433: U223.CO, U224.CI
- new net N$434: U223.DO, U224.DI
- new net N$435: U225.DO, U226.DI
- new net N$436: U225.CO, U226.CI
- new net N$437: U226.CO, U227.CI
- new net N$438: U226.DO, U227.DI
- new net N$439: U227.DO, U228.DI
- new net N$440: U227.CO, U228.CI
- new net N$441: U228.CO, U229.CI
- new net N$442: U228.DO, U229.DI
- new net N$443: U229.CO, U230.CI
- new net N$444: U229.DO, U230.DI
- new net N$445: U230.CO, U231.CI
- new net N$446: U230.DO, U231.DI
- new net N$447: U232.DO, U233.DI
- new net N$448: U232.CO, U233.CI
- new net N$449: U233.CO, U234.CI
- new net N$450: U233.DO, U234.DI
- new net N$451: U234.DO, U235.DI
- new net N$452: U234.CO, U235.CI
- new net N$453: U235.CO, U236.CI
- new net N$454: U235.DO, U236.DI
- new net N$455: U236.CO, U237.CI
- new net N$456: U236.DO, U237.DI
- new net N$457: U237.CO, U238.CI
- new net N$458: U237.DO, U238.DI
- new net N$459: U231.DO, U232.DI
- new net N$460: U231.CO, U232.CI
- new net N$461: U239.DO, U240.DI
- new net N$462: U239.CO, U240.CI
- new net N$463: U240.CO, U241.CI
- new net N$464: U240.DO, U241.DI
- new net N$465: U241.DO, U242.DI
- new net N$466: U241.CO, U242.CI
- new net N$467: U242.CO, U243.CI
- new net N$468: U242.DO, U243.DI
- new net N$469: U243.CO, U244.CI
- new net N$470: U243.DO, U244.DI
- new net N$471: U244.CO, U245.CI
- new net N$472: U244.DO, U245.DI
- new net N$473: U245.DO, U246.DI
- new net N$474: U245.CO, U246.CI
- new net N$475: U238.DO, U239.DI
- new net N$476: U238.CO, U239.CI
- new net N$477: U247.DI
- new net N$478: U247.CI
- new net N$479: U247.CO, U248.CI
- new net N$480: U247.DO, U248.DI
- new net N$481: U248.DO, U249.DI
- new net N$482: U248.CO, U249.CI
- new net N$483: U249.CO, U250.CI
- new net N$484: U249.DO, U250.DI
- new net N$485: U250.CO, U251.CI
- new net N$486: U250.DO, U251.DI
- new net N$487: U251.CO, U252.CI
- new net N$488: U251.DO, U252.DI
- new net N$489: U127.CI
- new net N$490: J1.3, U126.DO
- new net N$491: J2.4, U252.CO
- new net N$492: J2.3, U252.DO
- new net SD7: U196.DO, U197.DI
- new net SD8: U224.DO, U225.DI
- net GND: now also J1.1, J2.1, U191.GND, U192.GND, U193.GND, U194.GND, U195.GND, U196.GND, U197.GND, U198.GND, U199.GND, U200.GND, U201.GND, U202.GND, U203.GND, U204.GND, U205.GND, U206.GND, U207.GND, U208.GND, U209.GND, U210.GND, U211.GND, U212.GND, U213.GND, U214.GND, U215.GND, U216.GND, U217.GND, U218.GND, U219.GND, U220.GND, U221.GND, U222.GND, U223.GND, U224.GND, U225.GND, U226.GND, U227.GND, U228.GND, U229.GND, U230.GND, U231.GND, U232.GND, U233.GND, U234.GND, U235.GND, U236.GND, U237.GND, U238.GND, U239.GND, U240.GND, U241.GND, U242.GND, U243.GND, U244.GND, U245.GND, U246.GND, U247.GND, U248.GND, U249.GND, U250.GND, U251.GND, U252.GND
- net N$269: no longer U126.DO
- net N$270: now also J1.4; no longer U127.CI
- net VCC: now also J1.2, J2.2, U191.VCC, U192.VCC, U193.VCC, U194.VCC, U195.VCC, U196.VCC, U197.VCC, U198.VCC, U199.VCC, U200.VCC, U201.VCC, U202.VCC, U203.VCC, U204.VCC, U205.VCC, U206.VCC, U207.VCC, U208.VCC, U209.VCC, U210.VCC, U211.VCC, U212.VCC, U213.VCC, U214.VCC, U215.VCC, U216.VCC, U217.VCC, U218.VCC, U219.VCC, U220.VCC, U221.VCC, U222.VCC, U223.VCC, U224.VCC, U225.VCC, U226.VCC, U227.VCC, U228.VCC, U229.VCC, U230.VCC, U231.VCC, U232.VCC, U233.VCC, U234.VCC, U235.VCC, U236.VCC, U237.VCC, U238.VCC, U239.VCC, U240.VCC, U241.VCC, U242.VCC, U243.VCC, U244.VCC, U245.VCC, U246.VCC, U247.VCC, U248.VCC, U249.VCC, U250.VCC, U251.VCC, U252.VCC

Commit message: Laid out most of board
Connections:
- removed net N$491: J2.4, U252.CO
- removed net N$492: J2.3, U252.DO
- net N$269: now also J1.3
- net N$270: now also J2.3, U1.DI; no longer J1.4, U126.CO
- net N$423: now also U218.CO, U219.CI; no longer U219.DI
- net N$424: now also U218.DO, U219.DI; no longer U219.CI
- net N$477: now also U246.CO, U247.CI; no longer U247.DI
- net N$478: now also U246.DO, U247.DI; no longer U247.CI
- net N$489: now also J1.4
- net N$490: now also J2.4, U1.CI; no longer J1.3, U126.DO
Other:
- moved on the sheet: J1
Changed lines of the file:
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@@
 <part name="GND252" library="SparkFun-PowerSymbols" deviceset="GND" device=""/>
 <part name="J1" library="SparkFun-Connectors" deviceset="QWIIC_CONNECTOR" device="JS-1MM"/>
-<part name="SUPPLY253" library="SparkFun-PowerSymbols" deviceset="VCC" device=""/>
-<part name="GND253" library="SparkFun-PowerSymbols" deviceset="GND" device=""/>
 <part name="J2" library="SparkFun-Connectors" deviceset="QWIIC_CONNECTOR" device="JS-1MM"/>
-<part name="SUPPLY254" library="SparkFun-PowerSymbols" deviceset="VCC" device=""/>
-<part name="GND254" library="SparkFun-PowerSymbols" deviceset="GND" device=""/>
 </parts>
 <sheets>
@@
 <instance part="SUPPLY28" gate="G$1" x="205.74" y="63.5"/>
 <instance part="GND28" gate="1" x="205.74" y="43.18"/>
+<instance part="J2" gate="G$1" x="10.16" y="162.56"/>
 </instances>
 <busses>
@@
 <wire x1="20.32" y1="175.26" x2="20.32" y2="162.56" width="0.1524" layer="91"/>
 <wire x1="20.32" y1="162.56" x2="25.4" y2="162.56" width="0.1524" layer="91"/>
+<pinref part="J2" gate="G$1" pin="2"/>
+<wire x1="17.78" y1="162.56" x2="20.32" y2="162.56" width="0.1524" layer="91"/>
+<junction x="20.32" y="162.56"/>
 </segment>
 <segment>
@@
 <wire x1="20.32" y1="157.48" x2="20.32" y2="160.02" width="0.1524" layer="91"/>
 <wire x1="20.32" y1="160.02" x2="25.4" y2="160.02" width="0.1524" layer="91"/>
+<pinref part="J2" gate="G$1" pin="1"/>
+<wire x1="17.78" y1="160.02" x2="20.32" y2="160.02" width="0.1524" layer="91"/>
+<junction x="20.32" y="160.02"/>
 </segment>
 <segment>
@@
 </segment>
 </net>
+<net name="N$270" class="0">
+<segment>
+<pinref part="J2" gate="G$1" pin="3"/>
+<pinref part="U1" gate="G$1" pin="DI"/>
+<wire x1="17.78" y1="165.1" x2="25.4" y2="165.1" width="0.1524" layer="91"/>
+</segment>
+</net>
+<net name="N$490" class="0">
+<segment>
+<pinref part="J2" gate="G$1" pin="4"/>
+<pinref part="U1" gate="G$1" pin="CI"/>
+<wire x1="17.78" y1="167.64" x2="25.4" y2="167.64" width="0.1524" layer="91"/>
+</segment>
+</net>
 </nets>
 </sheet>
@@
 <instance part="SUPPLY140" gate="G$1" x="205.74" y="63.5"/>
 <instance part="GND140" gate="1" x="205.74" y="43.18"/>
-<instance part="J1" gate="G$1" x="243.84" y="124.46" rot="MR0"/>
-<instance part="SUPPLY253" gate="G$1" x="233.68" y="137.16"/>
-<instance part="GND253" gate="1" x="233.68" y="116.84"/>
+<instance part="J1" gate="G$1" x="10.16" y="88.9"/>
 </instances>
 <busses>
@@
 <wire x1="20.32" y1="101.6" x2="20.32" y2="88.9" width="0.1524" layer="91"/>
 <wire x1="20.32" y1="88.9" x2="25.4" y2="88.9" width="0.1524" layer="91"/>
+<pinref part="J1" gate="G$1" pin="2"/>
+<wire x1="17.78" y1="88.9" x2="20.32" y2="88.9" width="0.1524" layer="91"/>
+<junction x="20.32" y="88.9"/>
 </segment>
 <segment>
@@
 <wire x1="205.74" y1="50.8" x2="208.28" y2="50.8" width="0.1524" layer="91"/>
 </segment>
-<segment>
-<pinref part="SUPPLY253" gate="G$1" pin="VCC"/>
-<pinref part="J1" gate="G$1" pin="2"/>
-<wire x1="233.68" y1="137.16" x2="233.68" y2="124.46" width="0.1524" layer="91"/>
-<wire x1="233.68" y1="124.46" x2="236.22" y2="124.46" width="0.1524" layer="91"/>
-</segment>
 </net>
 <net name="GND" class="0">
@@
 <wire x1="20.32" y1="83.82" x2="20.32" y2="86.36" width="0.1524" layer="91"/>
 <wire x1="20.32" y1="86.36" x2="25.4" y2="86.36" width="0.1524" layer="91"/>
+<pinref part="J1" gate="G$1" pin="1"/>
+<wire x1="17.78" y1="86.36" x2="20.32" y2="86.36" width="0.1524" layer="91"/>
+<junction x="20.32" y="86.36"/>
 </segment>
 <segment>
@@
 <wire x1="205.74" y1="48.26" x2="208.28" y2="48.26" width="0.1524" layer="91"/>
 </segment>
-<segment>
-<pinref part="GND253" gate="1" pin="GND"/>
-<pinref part="J1" gate="G$1" pin="1"/>
-<wire x1="233.68" y1="119.38" x2="233.68" y2="121.92" width="0.1524" layer="91"/>
-<wire x1="233.68" y1="121.92" x2="236.22" y2="121.92" width="0.1524" layer="91"/>
-</segment>
 </net>
 <net name="N$217" class="0">
@@
 <pinref part="U127" gate="G$1" pin="DI"/>
 <wire x1="17.78" y1="91.44" x2="25.4" y2="91.44" width="0.1524" layer="91"/>
-</segment>
-</net>
-<net name="N$270" class="0">
-<segment>
-<pinref part="U126" gate="G$1" pin="CO"/>
-<wire x1="236.22" y1="129.54" x2="233.68" y2="129.54" width="0.1524" layer="91"/>
-<pinref part="J1" gate="G$1" pin="4"/>
+<pinref part="J1" gate="G$1" pin="3"/>
 </segment>
 </net>
@@
 <pinref part="U127" gate="G$1" pin="CI"/>
 <wire x1="25.4" y1="93.98" x2="22.86" y2="93.98" width="0.1524" layer="91"/>
-</segment>
-</net>
-<net name="N$490" class="0">
-<segment>
-<pinref part="U126" gate="G$1" pin="DO"/>
-<wire x1="233.68" y1="127" x2="236.22" y2="127" width="0.1524" layer="91"/>
-<pinref part="J1" gate="G$1" pin="3"/>
+<pinref part="J1" gate="G$1" pin="4"/>
+<wire x1="17.78" y1="93.98" x2="25.4" y2="93.98" width="0.1524" layer="91"/>
+<junction x="25.4" y="93.98"/>
 </segment>
 </net>
@@
 <net name="N$365" class="0">
 <segment>
-<pinref part="U190" gate="G$1" pin="CO"/>
-<pinref part="U191" gate="G$1" pin="CI"/>
-<wire x1="50.8" y1="55.88" x2="55.88" y2="55.88" width="0.1524" layer="91"/>
+<pinref part="U190" gate="G$1" pin="DO"/>
+<pinref part="U191" gate="G$1" pin="DI"/>
+<wire x1="50.8" y1="53.34" x2="55.88" y2="53.34" width="0.1524" layer="91"/>
 </segment>
 </net>
 <net name="N$366" class="0">
 <segment>
-<pinref part="U191" gate="G$1" pin="DI"/>
-<pinref part="U190" gate="G$1" pin="DO"/>
-<wire x1="55.88" y1="53.34" x2="50.8" y2="53.34" width="0.1524" layer="91"/>
+<pinref part="U190" gate="G$1" pin="CO"/>
+<pinref part="U191" gate="G$1" pin="CI"/>
+<wire x1="50.8" y1="55.88" x2="55.88" y2="55.88" width="0.1524" layer="91"/>
 </segment>
 </net>
@@
 </segment>
 </net>
-<net name="N$423" class="0">
-<segment>
-<pinref part="U219" gate="G$1" pin="DI"/>
-<wire x1="38.1" y1="15.24" x2="43.18" y2="15.24" width="0.1524" layer="91"/>
-</segment>
-</net>
-<net name="N$424" class="0">
-<segment>
-<pinref part="U219" gate="G$1" pin="CI"/>
-<wire x1="38.1" y1="17.78" x2="43.18" y2="17.78" width="0.1524" layer="91"/>
-</segment>
-</net>
-<net name="N$425" class="0">
-<segment>
-<pinref part="U219" gate="G$1" pin="CO"/>
-<pinref part="U220" gate="G$1" pin="CI"/>
-<wire x1="68.58" y1="17.78" x2="73.66" y2="17.78" width="0.1524" layer="91"/>
-</segment>
-</net>
-<net name="N$426" class="0">
-<segment>
-<pinref part="U219" gate="G$1" pin="DO"/>
-<pinref part="U220" gate="G$1" pin="DI"/>
-<wire x1="68.58" y1="15.24" x2="73.66" y2="15.24" width="0.1524" layer="91"/>
-</segment>
-</net>
 <net name="N$427" class="0">
 <segment>
@@
 </segment>
 </net>
+<net name="N$425" class="0">
+<segment>
+<pinref part="U219" gate="G$1" pin="CO"/>
+<pinref part="U220" gate="G$1" pin="CI"/>
+<wire x1="68.58" y1="17.78" x2="73.66" y2="17.78" width="0.1524" layer="91"/>
+</segment>
+</net>
+<net name="N$426" class="0">
+<segment>
+<pinref part="U220" gate="G$1" pin="DI"/>
+<pinref part="U219" gate="G$1" pin="DO"/>
+<wire x1="73.66" y1="15.24" x2="68.58" y2="15.24" width="0.1524" layer="91"/>
+</segment>
+</net>
+<net name="N$423" class="0">
+<segment>
+<pinref part="U218" gate="G$1" pin="CO"/>
+<pinref part="U219" gate="G$1" pin="CI"/>
+<wire x1="38.1" y1="17.78" x2="43.18" y2="17.78" width="0.1524" layer="91"/>
+</segment>
+</net>
+<net name="N$424" class="0">
+<segment>
+<pinref part="U219" gate="G$1" pin="DI"/>
+<pinref part="U218" gate="G$1" pin="DO"/>
+<wire x1="43.18" y1="15.24" x2="38.1" y2="15.24" width="0.1524" layer="91"/>
+</segment>
+</net>
 </nets>
 </sheet>
@@
 <instance part="SUPPLY252" gate="G$1" x="190.5" y="25.4"/>
 <instance part="GND252" gate="1" x="190.5" y="5.08"/>
-<instance part="J2" gate="G$1" x="231.14" y="12.7" rot="MR0"/>
-<instance part="SUPPLY254" gate="G$1" x="220.98" y="25.4"/>
-<instance part="GND254" gate="1" x="220.98" y="5.08"/>
 </instances>
 <busses>
@@
 <wire x1="190.5" y1="12.7" x2="193.04" y2="12.7" width="0.1524" layer="91"/>
 </segment>
-<segment>
-<pinref part="J2" gate="G$1" pin="2"/>
-<pinref part="SUPPLY254" gate="G$1" pin="VCC"/>
-<wire x1="223.52" y1="12.7" x2="220.98" y2="12.7" width="0.1524" layer="91"/>
-<wire x1="220.98" y1="12.7" x2="220.98" y2="25.4" width="0.1524" layer="91"/>
-</segment>
 </net>
 <net name="GND" class="0">
@@
 <wire x1="190.5" y1="10.16" x2="193.04" y2="10.16" width="0.1524" layer="91"/>
 </segment>
-<segment>
-<pinref part="GND254" gate="1" pin="GND"/>
-<pinref part="J2" gate="G$1" pin="1"/>
-<wire x1="220.98" y1="7.62" x2="220.98" y2="10.16" width="0.1524" layer="91"/>
-<wire x1="220.98" y1="10.16" x2="223.52" y2="10.16" width="0.1524" layer="91"/>
-</segment>
 </net>
 <net name="N$435" class="0">
@@
 </segment>
 </net>
-<net name="N$477" class="0">
-<segment>
-<pinref part="U247" gate="G$1" pin="DI"/>
-<wire x1="35.56" y1="15.24" x2="40.64" y2="15.24" width="0.1524" layer="91"/>
-</segment>
-</net>
-<net name="N$478" class="0">
-<segment>
-<pinref part="U247" gate="G$1" pin="CI"/>
-<wire x1="35.56" y1="17.78" x2="40.64" y2="17.78" width="0.1524" layer="91"/>
-</segment>
-</net>
 <net name="N$479" class="0">
 <segment>
@@
 </segment>
 </net>
-<net name="N$491" class="0">
+<net name="N$477" class="0">
 <segment>
-<pinref part="U252" gate="G$1" pin="CO"/>
-<wire x1="218.44" y1="17.78" x2="223.52" y2="17.78" width="0.1524" layer="91"/>
-<pinref part="J2" gate="G$1" pin="4"/>
+<pinref part="U246" gate="G$1" pin="CO"/>
+<pinref part="U247" gate="G$1" pin="CI"/>
+<wire x1="35.56" y1="17.78" x2="40.64" y2="17.78" width="0.1524" layer="91"/>
 </segment>
 </net>
-<net name="N$492" class="0">
+<net name="N$478" class="0">
 <segment>
-<pinref part="U252" gate="G$1" pin="DO"/>
-<wire x1="218.44" y1="15.24" x2="223.52" y2="15.24" width="0.1524" layer="91"/>
-<pinref part="J2" gate="G$1" pin="3"/>
+<pinref part="U246" gate="G$1" pin="DO"/>
+<pinref part="U247" gate="G$1" pin="DI"/>
+<wire x1="35.56" y1="15.24" x2="40.64" y2="15.24" width="0.1524" layer="91"/>
 </segment>
 </net>

Commit message: ordered v01
Parts:
- added FD1, FD2: FIDUCIALUFIDUCIAL, SparkFun-Aesthetics:FIDUCIALUFIDUCIAL
Connections:
- new net N$181: U95.DO, U96.DI
- new net N$182: U95.CO, U96.CI
Changed lines of the file:
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@@
 <part name="J1" library="SparkFun-Connectors" deviceset="QWIIC_CONNECTOR" device="JS-1MM"/>
 <part name="J2" library="SparkFun-Connectors" deviceset="QWIIC_CONNECTOR" device="JS-1MM"/>
+<part name="FD1" library="SparkFun-Aesthetics" deviceset="FIDUCIAL" device="UFIDUCIAL"/>
+<part name="FD2" library="SparkFun-Aesthetics" deviceset="FIDUCIAL" device="UFIDUCIAL"/>
 </parts>
 <sheets>
@@
 <instance part="GND28" gate="1" x="205.74" y="43.18"/>
 <instance part="J2" gate="G$1" x="10.16" y="162.56"/>
+<instance part="FD1" gate="G$1" x="228.6" y="30.48"/>
+<instance part="FD2" gate="G$1" x="231.14" y="30.48"/>
 </instances>
 <busses>
@@
 </segment>
 </net>
+<net name="N$181" class="0">
+<segment>
+<pinref part="U96" gate="G$1" pin="DI"/>
+<pinref part="U95" gate="G$1" pin="DO"/>
+<wire x1="147.32" y1="127" x2="142.24" y2="127" width="0.1524" layer="91"/>
+</segment>
+</net>
+<net name="N$182" class="0">
+<segment>
+<pinref part="U95" gate="G$1" pin="CO"/>
+<pinref part="U96" gate="G$1" pin="CI"/>
+<wire x1="142.24" y1="129.54" x2="147.32" y2="129.54" width="0.1524" layer="91"/>
+</segment>
+</net>
