File: Boards/Shield/ESP32Shield.sch (EAGLE design)
At the start: 25 parts, among them Q1 220mA/50V/3.5Ω, U1 5V

Commit message: updating shield
Parts:
- J1: device SparkFun-Connectors:CONN_16 -> SparkFun-Connectors:CONN_161X16_NO_SILK
- J7: device SparkFun-Connectors:CONN_12 -> SparkFun-Connectors:CONN_12NO_SILK
- LEFTEYE, RIGHTEYE: device SparkFun-Connectors:CONN_04 -> SparkFun-Connectors:CONN_041X04_NO_SILK
Connections:
- removed net 14: J7.10
- removed net 16: J1.14
- removed net 17: J1.15
- removed net 23: J1.16
- removed net 27: J7.6
- removed net 32: J7.9
- removed net 33: J7.7
- removed net BTN1: R36.2, S3.1
- removed net BTN2: R8.2, S1.SW-
- removed net CL: LEFTEYE.3, RIGHTEYE.3
- removed net DL: LEFTEYE.4
- removed net DR: RIGHTEYE.4
- removed net ENC-A: S1.A
- removed net ENC-B: S1.B
- removed net VUSB: J7.3
- new net 14/ENC-B: J7.10, S1.B
- new net 16/CLOCK: J1.14, LEFTEYE.3, RIGHTEYE.3
- new net 17/DR: J1.15, LEFTEYE.4
- new net 23/DL: J1.16, RIGHTEYE.4
- new net 27/BTN1: J7.6, R36.2, S3.1
- new net 32/ENC-A: J7.9, S1.A
- new net 33/BTN2: J7.7, R8.2, S1.SW-
- net 5V: now also J7.3, LEFTEYE.1, RIGHTEYE.1; no longer LEFTEYE.2, RIGHTEYE.2
- net GND: now also LEFTEYE.2, RIGHTEYE.2; no longer LEFTEYE.1, RIGHTEYE.1

Commit message: updating board to V06, finangling code to work with WROOM
Parts:
- removed C4: 1mF, SparkFun-Capacitors:1000UF-RADIAL-5MM-25V-20%
Connections:
- removed net 14/ENC-B: J7.10, S1.B
- removed net 32/ENC-A: J7.9, S1.A
- removed net 3V3: J1.2
- new net 14/ENC-A: J7.10, S1.A
- new net 32/ENC-B: J7.9, S1.B
- net 3.3V: now also J1.2
- net 5V: no longer C4.+
- net GND: no longer C4.-
Changed lines of the file:
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@@
 <?xml version="1.0" encoding="utf-8"?>
 <!DOCTYPE eagle SYSTEM "eagle.dtd">
-<eagle version="9.1.0">
+<eagle version="9.1.3">
 <drawing>
 <settings>
@@
 <part name="U1" library="SparkFun-IC-Power" deviceset="V_REG_MIC5205" device="5V" value="5V"/>
 <part name="GND2" library="SparkFun-PowerSymbols" deviceset="GND" device=""/>
-<part name="C4" library="SparkFun-Capacitors" deviceset="1000UF" device="-RADIAL-5MM-25V-20%" value="1mF"/>
-<part name="GND4" library="SparkFun-PowerSymbols" deviceset="GND" device=""/>
-<part name="SUPPLY1" library="SparkFun-PowerSymbols" deviceset="5V" device=""/>
 <part name="SUPPLY2" library="SparkFun-PowerSymbols" deviceset="5V" device=""/>
 <part name="SUPPLY3" library="SparkFun-PowerSymbols" deviceset="5V" device=""/>
@@
 <part name="J7" library="SparkFun-Connectors" deviceset="CONN_12" device="NO_SILK"/>
 <part name="SUPPLY7" library="SparkFun-PowerSymbols" deviceset="5V" device=""/>
+<part name="SUPPLY8" library="SparkFun-PowerSymbols" deviceset="3.3V" device=""/>
 </parts>
 <sheets>
@@
 <instance part="U1" gate="U1" x="193.04" y="157.48"/>
 <instance part="GND2" gate="1" x="180.34" y="144.78"/>
-<instance part="C4" gate="G$1" x="12.7" y="88.9"/>
-<instance part="GND4" gate="1" x="12.7" y="78.74"/>
-<instance part="SUPPLY1" gate="G$1" x="12.7" y="96.52"/>
 <instance part="SUPPLY2" gate="G$1" x="231.14" y="137.16"/>
 <instance part="SUPPLY3" gate="G$1" x="20.32" y="22.86"/>
@@
 <instance part="J7" gate="G$1" x="45.72" y="129.54" rot="MR0"/>
 <instance part="SUPPLY7" gate="G$1" x="33.02" y="144.78"/>
+<instance part="SUPPLY8" gate="G$1" x="68.58" y="109.22"/>
 </instances>
 <busses>
@@
 </segment>
 <segment>
-<pinref part="C4" gate="G$1" pin="-"/>
-<wire x1="12.7" y1="83.82" x2="12.7" y2="81.28" width="0.1524" layer="91"/>
-<pinref part="GND4" gate="1" pin="GND"/>
-</segment>
-<segment>
 <pinref part="GND6" gate="1" pin="GND"/>
 <pinref part="J4" gate="G$1" pin="1"/>
@@
 </net>
 <net name="5V" class="0">
-<segment>
-<pinref part="C4" gate="G$1" pin="+"/>
-<wire x1="12.7" y1="91.44" x2="12.7" y2="96.52" width="0.1524" layer="91"/>
-<pinref part="SUPPLY1" gate="G$1" pin="5V"/>
-</segment>
 <segment>
 <wire x1="20.32" y1="15.24" x2="20.32" y2="22.86" width="0.1524" layer="91"/>
@@
 <pinref part="SUPPLY6" gate="G$1" pin="3.3V"/>
 </segment>
-</net>
-<net name="32/ENC-A" class="0">
-<segment>
-<pinref part="S1" gate="G$1" pin="A"/>
-<wire x1="132.08" y1="38.1" x2="137.16" y2="38.1" width="0.1524" layer="91"/>
-<label x="137.16" y="38.1" size="1.27" layer="95" font="vector" xref="yes"/>
-</segment>
-<segment>
-<pinref part="J7" gate="G$1" pin="9"/>
-<wire x1="35.56" y1="134.62" x2="30.48" y2="134.62" width="0.1524" layer="91"/>
-<label x="30.48" y="134.62" size="1.27" layer="95" font="vector" rot="R180" xref="yes"/>
-<label x="30.48" y="134.62" size="1.27" layer="95" font="vector" rot="R180" xref="yes"/>
-</segment>
-</net>
-<net name="14/ENC-B" class="0">
-<segment>
-<pinref part="S1" gate="G$1" pin="B"/>
-<wire x1="132.08" y1="48.26" x2="137.16" y2="48.26" width="0.1524" layer="91"/>
-<label x="137.16" y="48.26" size="1.27" layer="95" font="vector" xref="yes"/>
-</segment>
-<segment>
-<pinref part="J7" gate="G$1" pin="10"/>
-<wire x1="35.56" y1="137.16" x2="30.48" y2="137.16" width="0.1524" layer="91"/>
-<label x="30.48" y="137.16" size="1.27" layer="95" font="vector" rot="R180" xref="yes"/>
+<segment>
+<pinref part="J1" gate="G$1" pin="2"/>
+<wire x1="55.88" y1="106.68" x2="68.58" y2="106.68" width="0.1524" layer="91"/>
+<pinref part="SUPPLY8" gate="G$1" pin="3.3V"/>
+<wire x1="68.58" y1="109.22" x2="68.58" y2="106.68" width="0.1524" layer="91"/>
 </segment>
 </net>
@@
 </segment>
 </net>
-<net name="3V3" class="0">
-<segment>
-<pinref part="J1" gate="G$1" pin="2"/>
-<wire x1="55.88" y1="106.68" x2="58.42" y2="106.68" width="0.1524" layer="91"/>
-<label x="58.42" y="106.68" size="1.27" layer="95" font="vector" xref="yes"/>
-</segment>
-</net>
 <net name="NC" class="0">
 <segment>
@@
 </segment>
 </net>
+<net name="14/ENC-A" class="0">
+<segment>
+<pinref part="J7" gate="G$1" pin="10"/>
+<wire x1="35.56" y1="137.16" x2="30.48" y2="137.16" width="0.1524" layer="91"/>
+<label x="30.48" y="137.16" size="1.27" layer="95" font="vector" rot="R180" xref="yes"/>
+</segment>
+<segment>
+<pinref part="S1" gate="G$1" pin="A"/>
+<wire x1="132.08" y1="38.1" x2="137.16" y2="38.1" width="0.1524" layer="91"/>
+<label x="137.16" y="38.1" size="1.27" layer="95" font="vector" xref="yes"/>
+</segment>
+</net>
+<net name="32/ENC-B" class="0">
+<segment>
+<pinref part="J7" gate="G$1" pin="9"/>
+<wire x1="35.56" y1="134.62" x2="30.48" y2="134.62" width="0.1524" layer="91"/>
+<label x="30.48" y="134.62" size="1.27" layer="95" font="vector" rot="R180" xref="yes"/>
+<label x="30.48" y="134.62" size="1.27" layer="95" font="vector" rot="R180" xref="yes"/>
+</segment>
+<segment>
+<pinref part="S1" gate="G$1" pin="B"/>
+<wire x1="132.08" y1="48.26" x2="137.16" y2="48.26" width="0.1524" layer="91"/>
+<label x="137.16" y="48.26" size="1.27" layer="95" font="vector" xref="yes"/>
+</segment>
+</net>
